File: HW/KicadProject/MIDIPresetController.kicad_pcb (KiCad board)
At the start: 2 copper layers, 40 x 75 mm, 25 parts, among them J1 Conn_01x02, J2 Conn_01x03, J3 Conn_02x05_Odd_Even, J4 Conn_01x02, J5 Conn_01x02, SW1 SW_SPST, SW2 SW_DIP_x04, U1 74LVC1G34, U2 STM32L011D4Px

Commit message: Updated to kicad 7.0.1, added stm32 doc links into schema page, regen pdf schema
Connections:
- U1 pad 1: (no net) -> unconnected-(U1-NC-Pad1)
